File: bambu-lab-xa007.kicad_sch (KiCad schematic)
At the start: 4 parts, among them J1 Side_B, J2 Side_A, SW1 SW_SPDT

Commit message: fix: modify footprint for mounting hole to be M2.5
Parts:
- H1: footprint MountingHole:MountingHole_2.5mm_Pad -> MountingHole:MountingHole_2.7mm_M2.5_Pad_TopBottom
Changed lines of the file:
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@@
 			)
 		)
-		(property "Footprint" "MountingHole:MountingHole_2.5mm_Pad"
+		(property "Footprint" "MountingHole:MountingHole_2.7mm_M2.5_Pad_TopBottom"
 			(at 123.19 108.585 0)
 			(effects
